File: allwinner_v3s_1.kicad_pcb (KiCad board)
At the start: 4 copper layers, 100.2 x 55.7 mm, 236 parts, among them IC1 SX1250IMLTRT, IC2 SX1250IMLTRT, IC4 SX1302IMLTRT, J1 Conn_Coaxial, J2 Conn_01x03_Pin, J3 RJ45_Hanrun_HR911105A_Horizon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, J5 USB_C_Receptacle_USB2.0_16P, J6 Conn_01x07_Pin, SW1 KMR731NG LFS, U1 AllwinnerV3S, U10 BMI-S-205-C, U11 SDG02GWSIGA-CSNP2, U2 L86M33, U3 TPS62132, U4 TPS62130, U5 ESD701DPYR, U6 TPS62131, U7 TPS62130, U8 TPS7A2033PDBVR, U9 SKY66420-11, Y1 TX21-M010S-32.000-X-R, Y2 ABS07-32.768KHZ-7-T, Y3 ABM8-24.000MHZ-B2-T

Commit message: The ___  invisible ghost gerber curve trace deleted :)
Parts:
- moved U10 0.10 mm to (86.0, 72.6)
Routing:
- net 3V3: track 65.6 -> 64.2 mm
- net +3V: track 85.2 -> 84.0 mm
- net +1V8: track 98.3 -> 99.4 mm
- net +1V2: track 192.8 -> 192.2 mm
Other:
- outline, holes or cut-outs redrawn
